Commit message: implementation of moveit

File: src/robot_description/urdf/robot.urdf.xacro (robot description, xacro)
@@ -1,4 +1,6 @@
 <?xml version="1.0"?>
-<robot xmlns:xacro="https://www.ros.org/wiki/xacro" name="arduinobot">
+<robot xmlns:xacro="https://www.ros.org/wiki/xacro" name="pibot">
+    <!-- <xacro:include filename="$(find robot_description)/urdf/robot_gazebo.xacro"/> -->
+    <xacro:include filename="$(find robot_description)/urdf/robot_ros2_control.xacro"/>
     <xacro:property name="effort_big_servo" value="1.32" />
     <xacro:property name="velocity_big_servo" value="6.16" />
@@ -15,10 +17,10 @@
             </material>
         </visual>
-        <collision>
+        <!-- <collision>
             <origin rpy="0 0 0" xyz="0 0 0"/>
                 <geometry>
                     <mesh filename="package://robot_description/meshes/Base_Bottom.stl" scale="0.01 0.01 0.01"/>
                 </geometry>
-        </collision>
+        </collision> -->
         <inertial>
             <mass value="0.312"/>
@@ -41,10 +43,10 @@
             </material>
         </visual>
-        <collision>
+        <!-- <collision>
             <origin rpy="0 0 0" xyz="0 0 0"/>
             <geometry>
                 <mesh filename="package://robot_description/meshes/Base_Plate_with_Servo.stl" scale="0.01 0.01 0.01"/>
             </geometry>
-        </collision>
+        </collision> -->
         <inertial>
             <mass value="0.135"/>
@@ -61,5 +63,5 @@
     <link name="first_arm">
         <visual>
-            <origin rpy="0 ${PI/2} 0" xyz="-0.1 -0.1 -0.33"/>
+            <origin rpy="0 ${-PI/2} 0" xyz="0.1 -0.1 -0.33"/>
             <geometry>
                 <mesh filename="package://robot_description/meshes/Joint_1_with_Servo.stl" scale="0.01 0.01 0.01"/>
@@ -69,10 +71,10 @@
             </material>
         </visual>
-        <collision>
-            <origin rpy="0 ${PI/2} 0" xyz="-0.1 -0.1 -0.33"/>
+        <!-- <collision>
+            <origin rpy="0 ${-PI/2} 0" xyz="-0.1 -0.1 -0.33"/>
             <geometry>
                 <mesh filename="package://robot_description/meshes/Joint_1_with_Servo.stl" scale="0.01 0.01 0.01"/>
             </geometry>
-        </collision>
+        </collision> -->
         <inertial>
             <mass value="0.070"/>
@@ -87,3 +89,114 @@
         <limit lower="-${PI/2}" upper="${PI/2}" effort="${effort_big_servo}" velocity="${velocity_big_servo}"/>
     </joint>
+    <link name="second_arm">
+        <visual>
+            <origin rpy="0 -${PI/2} 0" xyz="0.1 -0.1 -0.33"/>
+            <geometry>
+                <mesh filename="package://robot_description/meshes/SecondArm.stl" scale="0.01 0.01 0.01"/>
+            </geometry>
+            <material name="green">
+                <color rgba="0 1 0 1"/>
+            </material>
+        </visual>
+        <!-- <collision>
+            <origin rpy="0 -${PI/2} 0" xyz="0.1 -0.1 -0.33"/>
+            <geometry>
+                <mesh filename="package://robot_description/meshes/SecondArm.stl" scale="0.01 0.01 0.01"/>
+            </geometry>
+        </collision> -->
+        <inertial>
+            <mass value="0.070"/>
+            <inertia ixx="0.0002" ixy="0.0" ixz="0.0" iyy="0.0002" iyz="0.0" izz="0.0002"/>
+        </inertial>
+    </link>
+    <joint name="joint_3" type="revolute">
+        <parent link="first_arm"/>
+        <child link="second_arm"/>
+        <axis xyz="0 0 1"/>
+        <origin rpy="0 0 0" xyz="0 1.3 0"/>
+        <limit lower="-${PI/2}" upper="${PI/2}" effort="${effort_big_servo}" velocity="${velocity_big_servo}"/>
+    </joint>
+    <link name="gripper_base">
+        <visual>
+            <origin rpy="0 -${PI/2} ${PI}" xyz="-0.04 0.2 0.005"/>
+            <geometry>
+                <mesh filename="package://robot_description/meshes/GripperBase.stl" scale="0.01 0.01 0.01"/>
+            </geometry>
+            <material name="green">
+                <color rgba="0 1 0 1"/>
+            </material>
+        </visual>
+        <!-- <collision>
+            <origin rpy="0 -${PI/2} ${PI}" xyz="-0.04 0.2 0.005"/>
+            <geometry>
+                <mesh filename="package://robot_description/meshes/GripperBase.stl" scale="0.01 0.01 0.01"/>
+            </geometry>
+        </collision> -->
+        <inertial>
+            <mass value="0.070"/>
+            <inertia ixx="0.0002" ixy="0.0" ixz="0.0" iyy="0.0002" iyz="0.0" izz="0.0002"/>
+        </inertial>
+    </link>
+    <joint name="joint_4_fixed_gripper" type="fixed">
+        <parent link="second_arm"/>
+        <child link="gripper_base"/>
+        <origin rpy="0 0 0" xyz="-0.05 0.625 -0.33"/>
+    </joint>
+    <link name="gripper_right">
+        <visual>
+            <origin rpy="0 0 0" xyz="0 0 0"/>
+            <geometry>
+                <mesh filename="package://robot_description/meshes/GripperRightFinger.stl" scale="0.01 0.01 0.01"/>
+            </geometry>
+            <material name="green">
+                <color rgba="0 1 0 1"/>
+            </material>
+        </visual>
+        <!-- <collision>
+            <origin rpy="0 0 0" xyz="0 0 0"/>
+            <geometry>
+                <mesh filename="package://robot_description/meshes/GripperRightFinger.stl" scale="0.01 0.01 0.01"/>
+            </geometry>
+        </collision> -->
+        <inertial>
+            <mass value="0.070"/>
+            <inertia ixx="0.0002" ixy="0.0" ixz="0.0" iyy="0.0002" iyz="0.0" izz="0.0002"/>
+        </inertial>
+    </link>
+    <joint name="gripper" type="revolute">
+        <parent link="gripper_base"/>
+        <child link="gripper_right"/>
+        <axis xyz="0 0 1"/>
+        <origin rpy="0 ${PI/2} 0" xyz="0 0.2 -0.05"/>
+        <limit lower="-${PI/2}" upper="${PI/2}" effort="${effort_big_servo}" velocity="${velocity_big_servo}"/>
+    </joint>
+    <link name="gripper_left">
+        <visual>
+            <origin rpy="0 0 ${196 * PI/180}" xyz="0 0 0"/>
+            <geometry>
+                <mesh filename="package://robot_description/meshes/GripperLeftFinger.stl" scale="0.01 0.01 0.01"/>
+            </geometry>
+            <material name="green">
+                <color rgba="0 1 0 1"/>
+            </material>
+        </visual>
+        <!-- <collision>
+            <origin rpy="0 0 ${196 * PI/180}" xyz="0 0 0"/>
+            <geometry>
+                <mesh filename="package://robot_description/meshes/GripperLeftFinger.stl" scale="0.01 0.01 0.01"/>
+            </geometry>
+        </collision> -->
+        <inertial>
+            <mass value="0.070"/>
+            <inertia ixx="0.0002" ixy="0.0" ixz="0.0" iyy="0.0002" iyz="0.0" izz="0.0002"/>
+        </inertial>
+    </link>
+    <joint name="gripper2" type="revolute">
+        <parent link="gripper_base"/>
+        <child link="gripper_left"/>
+        <axis xyz="0 0 1"/>
+        <origin rpy="0 ${PI/2} 0" xyz="0 0.2 0.1"/>
+        <limit lower="-${PI/2}" upper="${PI/2}" effort="${effort_big_servo}" velocity="${velocity_big_servo}"/>
+        <mimic joint="gripper" multiplier="-1" offset="0"/>
+    </joint>
 </robot>

Commit message: Implementation of the Sequence saving deleting and sending functionality in the GUI Window

File: src/robot_description/urdf/robot.urdf.xacro (robot description, xacro)
@@ -143,4 +143,16 @@
         <origin rpy="0 0 0" xyz="-0.05 0.625 -0.33"/>
     </joint>
+    <link name="ee_link">
+        <inertial>
+            <mass value="0.001"/>
+            <inertia ixx="1e-6" iyy="1e-6" izz="1e-6" ixy="0" ixz="0" iyz="0"/>
+        </inertial>
+    </link>
+    <joint name="ee_fixed_joint" type="fixed">
+        <parent link="gripper_base"/>
+        <child link="ee_link"/>
+        <!-- Mittelpunkt zwischen den Greiferbacken -->
+        <origin xyz="0 0.64 0.03" rpy="0 0 0"/>
+    </joint>
     <link name="gripper_right">
         <visual>

Commit message: docs: finalize README and synchronize robot visualization Completed README structure (demo video pending) Updated Rviz model colors to match the physical PI-Bot hardware Added system diagrams and assets to /docs Created requirements.txt for streamlined dependency installation

File: src/robot_description/urdf/robot.urdf.xacro (robot description, xacro)
@@ -14,5 +14,5 @@
                 </geometry>
             <material name="gray">
-                <color rgba="0.2 0.2 0.2 1"/>
+                <color rgba="0.0 0.0 0.0 1.0"/>
             </material>
         </visual>
@@ -40,5 +40,5 @@
             </geometry>
             <material name="black">
-                <color rgba="0 0 0 1.0"/>
+                <color rgba="0.0 0.0 0.0 1.0"/>
             </material>
         </visual>
@@ -67,6 +67,6 @@
                 <mesh filename="package://robot_description/meshes/Joint_1_with_Servo.stl" scale="0.01 0.01 0.01"/>
             </geometry>
-            <material name="green">
-                <color rgba="0 1 0 1"/>
+            <material name="dark_gray">
+                <color rgba="0.2 0.2 0.2 1.0"/>
             </material>
         </visual>
@@ -95,6 +95,6 @@
                 <mesh filename="package://robot_description/meshes/SecondArm.stl" scale="0.01 0.01 0.01"/>
             </geometry>
-            <material name="green">
-                <color rgba="0 1 0 1"/>
+            <material name="white">
+                <color rgba="1.0 1.0 1.0 1.0"/>
             </material>
         </visual>
@@ -114,5 +114,5 @@
         <child link="second_arm"/>
         <axis xyz="0 0 1"/>
-        <origin rpy="0 0 0" xyz="0 1.3 0"/>
+        <origin rpy="0 0 ${PI/2}" xyz="0 1.3 0"/>
         <limit lower="-${PI/2}" upper="${PI/2}" effort="${effort_big_servo}" velocity="${velocity_big_servo}"/>
     </joint>
@@ -123,6 +123,6 @@
                 <mesh filename="package://robot_description/meshes/GripperBase.stl" scale="0.01 0.01 0.01"/>
             </geometry>
-            <material name="green">
-                <color rgba="0 1 0 1"/>
+            <material name="white">
+                <color rgba="1.0 1.0 1.0 1.0"/>
             </material>
         </visual>
@@ -161,6 +161,6 @@
                 <mesh filename="package://robot_description/meshes/GripperRightFinger.stl" scale="0.01 0.01 0.01"/>
             </geometry>
-            <material name="green">
-                <color rgba="0 1 0 1"/>
+            <material name="blue">
+                <color rgba="0.2 0.4 1.0 1.0"/>
             </material>
         </visual>
@@ -189,6 +189,6 @@
                 <mesh filename="package://robot_description/meshes/GripperLeftFinger.stl" scale="0.01 0.01 0.01"/>
             </geometry>
-            <material name="green">
-                <color rgba="0 1 0 1"/>
+            <material name="red">
+                <color rgba="1.0 0.15 0.15 1.0"/>
             </material>
         </visual>

Commit message: - Updating the Quickstart instructions because while testing PySide6 was not found by ros therefore break system installation is required
- small change of starting pose of the robot

File: src/robot_description/urdf/robot.urdf.xacro (robot description, xacro)
@@ -114,5 +114,5 @@
         <child link="second_arm"/>
         <axis xyz="0 0 1"/>
-        <origin rpy="0 0 ${PI/2}" xyz="0 1.3 0"/>
+        <origin rpy="0 0 0" xyz="0 1.3 0"/>
         <limit lower="-${PI/2}" upper="${PI/2}" effort="${effort_big_servo}" velocity="${velocity_big_servo}"/>
     </joint>
